File: Simple_BLDC_Driver/Simple_BLDC_Driver.kicad_sch (KiCad schematic)
At the start: 0 parts

Commit message: start the shematic
Parts:
- added C1, C2, C3, C4, C5, C6: C_Polarized, Capacitor_THT:CP_Radial_D16.0mm_P7.50mm, symbol Device:C_Polarized
- added C11, C21, C22, C24, C25, C26, C27, C28, C29, C30, C31, C32, C33: 10u, Capacitor_SMD:C_0805_2012Metric, symbol Device:C
- added C17, C7, C8, C9: 100n, Capacitor_SMD:C_0805_2012Metric, symbol Device:C
- added C23: 1u, Capacitor_SMD:C_0805_2012Metric, symbol Device:C
- added C34, C35, C36: 10n, Capacitor_SMD:C_0805_2012Metric, symbol Device:C
- added D32: D_Schottky, Diode_SMD:D_SMA, symbol Device:D_Schottky
- added D4, D5, D6, D7, D8: YLED1206R, LED_SMD:LED_1206_3216Metric, symbol Device:LED
- added F1: Fuse, Fuse:Fuse_2512_6332Metric, symbol Device:Fuse
- added IC1, IC2, IC3: UCC27282DR, Package_SO:SOIC-8_3.9x4.9mm_P1.27mm, symbol UCC27282DR:UCC27282DR
- added J1: Conn_01x02, Connector_Phoenix_MC:PhoenixContact_MCV_1,5_2-G-3.5_1x02_P3.50mm_Vertical, symbol Connector_Generic:Conn_01x02
- added J2: Conn_01x03, Connector_Phoenix_MC:PhoenixContact_MCV_1,5_3-G-3.5_1x03_P3.50mm_Vertical, symbol Connector_Generic:Conn_01x03
- added JP1: SolderJumper_2_Bridged, Jumper:SolderJumper-2_P1.3mm_Bridged2Bar_RoundedPad1.0x1.5mm, symbol Jumper:SolderJumper_2_Bridged
- added L1: 12uH, Inductor_SMD:L_Coilcraft_XAL6020-XXX, symbol Device:L
- added Q1, Q2, Q3, Q4, Q5, Q6: Q_NMOS, Package_DFN_QFN:PQFN-8-EP_6x5mm_P1.27mm_Generic, symbol Device:Q_NMOS
- added R1, R2, R3, R4, R5, R6: 10R, Resistor_SMD:R_0805_2012Metric, symbol Device:R
- added R29, R30, R61: R, Resistor_SMD:R_0805_2012Metric, symbol Device:R
- added R34: 2K, Resistor_SMD:R_0805_2012Metric, symbol Device:R
- added R35, R36, R37, R38: 220R, Resistor_SMD:R_0805_2012Metric, symbol Device:R
- added R62, R63, R64, R65, R66, R67: 10k, Resistor_SMD:R_0805_2012Metric, symbol Device:R
- added U1: BP, Library:blue_pill, symbol New_Library:BP
- added U2: L7805, Package_TO_SOT_SMD:TO-252-2, symbol Regulator_Linear:L7805
- added U7: LV2842XLVDDCR, Package_TO_SOT_SMD:SOT-23-6, symbol Regulator_Switching:LV2862XDDC
Connections:
- new net: R36.1, U1.PB10
- new net: D7.2 (A), R36.2
- new net: C8.1, IC2.2 (HB)
- new net: C35.1, C8.2, IC2.4 (HS), J2.2 (Pin_2), Q3.S, Q4.D
- new net: R29.2, R30.1, R61.1, U7.3 (FB)
- new net: D8.2 (A), R35.2
- new net: C11.1, JP1.1 (A), U7.5 (VIN)
- new net: C34.1, C7.2, IC1.4 (HS), J2.1 (Pin_1), Q1.S, Q2.D
- new net: C36.1, C9.2, IC3.4 (HS), J2.3 (Pin_3), Q5.S, Q6.D
- new net: IC3.3 (HO), R5.1
- new net: Q5.G, R5.2
- new net: IC2.3 (HO), R3.1
- new net: IC2.8 (LO), R4.1
- new net: Q2.G, R2.2
- new net: Q3.G, R3.2
- new net: R38.1, U1.PB0
- new net: D5.2 (A), R38.2
- new net: Q6.G, R6.2
- new net: C7.1, IC1.2 (HB)
- new net: C17.1, U7.1 (CB)
- new net: C17.2, D32.1 (K), L1.1, U7.6 (SW)
- new net: IC1.3 (HO), R1.1
- new net: IC1.8 (LO), R2.1
- new net: F1.1, J1.2 (Pin_2)
- new net: C9.1, IC3.2 (HB)
- new net: IC3.8 (LO), R6.1
- new net: Q1.G, R1.2
- new net: Q4.G, R4.2
- new net: R37.1, U1.PB1
- new net: D6.2 (A), R37.2
- new net: D4.2 (A), R34.2
- new net: R35.1, U1.PB11
- new net +12V: C21.1, C23.1, C25.1, C28.1, C31.1, C5.1, IC1.1 (VDD), IC2.1 (VDD), IC3.1 (VDD), L1.2, R29.1, R34.1, U2.1 (IN)
- new net +24V: C1.1, C2.1, C26.1, C27.1, C29.1, C3.1, C30.1, C32.1, C33.1, C4.1, F1.2, JP1.2 (B), Q1.D, Q3.D, Q5.D
- new net +5V: C22.1, C24.1, C6.1, U1.5V, U2.3 (OUT)
- new net GND: C1.2, C11.2, C2.2, C21.2, C22.2, C23.2, C24.2, C25.2, C26.2, C27.2, C28.2, C29.2, C3.2, C30.2, C31.2, C32.2, C33.2, C34.2, C35.2, C36.2, C4.2, C5.2, C6.2, D32.2 (A), D4.1 (K), D5.1 (K), D6.1 (K), D7.1 (K), D8.1 (K), IC1.7 (VSS), IC2.7 (VSS), IC3.7 (VSS), J1.1 (Pin_1), Q2.S, Q4.S, Q6.S, R30.2, R61.2, R62.2, R63.2, R64.2, R65.2, R66.2, R67.2, U1.G (GND), U2.2 (GND), U7.2 (GND)
- new net H_A: IC1.5 (HI), R67.1, U1.PA8
- new net H_B: IC2.5 (HI), R66.1, U1.PA9
- new net H_C: IC3.5 (HI), R65.1, U1.PA10
- new net L_A: IC1.6 (LI), R62.1, U1.PB13
- new net L_B: IC2.6 (LI), R63.1, U1.PB14
- new net L_C: IC3.6 (LI), R64.1, U1.PB15
- no-connect marks 0 -> 1
Other:
- note added: "!!!"
- note added: "0.765V"
- note added: "12V"
- note added: "5V"
- note added: "MOTOR"
- note added: "POWER input"
- note added: "Phase A"
- note added: "Phase B"
- note added: "Phase C"
- note added: "power"
